File: 2017_Motherboard/Arduino_MEGA_2560-Rev3.brd (EAGLE design)
At the start: 100 x 80 mm, 86 parts, among them IC1 NCP1117ST50T3G, IC2 FT232RL, IC3 ATMEGA2560-16AU, IC7 LMV358IDGKR, X1 POWERSUPPLY_DC21MMX, Y1 CSTCE16M0V53-R0 16MHZ

Commit message: Reverted schematic and Layout
took out video and and added support for orientation sensor. schematic
and layout are in sync again
Parts:
- removed XIO: 18x2F-H8.5, SmartPrj:2X18
- added BLUETOOTH_J6, ESC_PWM_GND: (no value), SparkFun-Connectors:1X06_LONGPADS
- added IC4: MAX4312ESE, maxim:SO16
- added IC5: MAX3468CPA, maxim:DIL08
- added RXD2_JUMPER, TXD2_JUMPER: (no value), SparkFun-Connectors:1X02
- added VIDEO_IN, VIDEO_IN_GND: 8x1F-H8.5, SmartPrj:1X08
- added VIDEO_OUT: A1944-50, con-coax:A1944
- J12, J9: device SparkFun-Connectors:1X06_LONGPADS -> SparkFun-Connectors:1X13
- moved R30 436.7 mm to (2.29, 37.3), turned to 180 degrees
- moved D2 408.4 mm to (2.29, 39.4), turned to 90 degrees
- moved J11 375.8 mm to (10.2, 39.6), turned to 90 degrees
- moved J10 368.8 mm to (3.05, 53.3)
- moved J8 362.3 mm to (7.62, 74.9), turned to 90 degrees
- moved J7 320.8 mm to (30.2, 51.8), turned to 180 degrees
- moved J6 298.1 mm to (30.2, 49.3), turned to 180 degrees
- moved R19 281.5 mm to (24.9, 55.1), turned to 180 degrees
- moved R21 281.4 mm to (19.6, 57.1), turned to 180 degrees
- moved R24 278.6 mm to (16.0, 43.2)
- moved R18 273.2 mm to (24.9, 53.6), turned to 180 degrees
- moved R23 271.3 mm to (16.0, 41.7), turned to 180 degrees
- moved C17 270.9 mm to (15.2, 57.1)
- moved R22 270.3 mm to (16.0, 39.9)
- moved R20 269.3 mm to (16.0, 44.7)
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Connections:
- removed net INV: J1.6
- removed net RESET_B: R22.1
- new net RXD2_OUT: IC5.6, J13.2, RXD2_JUMPER.2
- new net TXD2_OUT: IC5.7, J13.1, TXD2_JUMPER.2
- new net VIDEO_OUT: IC4.16, VIDEO_OUT.1
- new net VID_0: IC4.5, VIDEO_IN.1
- new net VID_1: IC4.6, VIDEO_IN.2
- new net VID_2: IC4.7, VIDEO_IN.3
- new net VID_3: IC4.8, VIDEO_IN.4
- new net VID_4: IC4.9, VIDEO_IN.5
- new net VID_5: IC4.10, VIDEO_IN.6
- new net VID_6: IC4.11, VIDEO_IN.7
- new net VID_7: IC4.12, VIDEO_IN.8
- net +5V: now also BLUETOOTH_J6.2, IC4.4, IC5.8, J1.6, J12.13; no longer J12.2, XIO.1, XIO.2
- net GND: now also BLUETOOTH_J6.3, ESC_PWM_GND.1, ESC_PWM_GND.2, ESC_PWM_GND.3, ESC_PWM_GND.4, ESC_PWM_GND.5, ESC_PWM_GND.6, IC4.13, IC4.14, IC4.15, IC5.5, VIDEO_IN_GND.1, VIDEO_IN_GND.2, VIDEO_IN_GND.3, VIDEO_IN_GND.4, VIDEO_IN_GND.5, VIDEO_IN_GND.6, VIDEO_IN_GND.7, VIDEO_IN_GND.8, VIDEO_OUT.2, VIDEO_OUT.3, VIDEO_OUT.4, VIDEO_OUT.5; no longer J12.3, J9.2, J9.3, J9.4, J9.5, J9.6, XIO.35, XIO.36
- net PA0: no longer XIO.3
- net PA1: now also BLUETOOTH_J6.6; no longer J12.6, XIO.4
- net PA2: now also BLUETOOTH_J6.1; no longer J12.1, XIO.5
- net PA3: now also IC4.3; no longer XIO.6
- net PA4: now also IC4.2; no longer XIO.7
- net PA5: now also IC4.1; no longer XIO.8
- net PA6: now also IC5.2; no longer XIO.9
- net PA7: now also IC5.3; no longer XIO.10
- net PB0: now also J12.1; no longer XIO.34
- net PB1: now also J9.13; no longer XIO.33
- net PB2: now also J12.2; no longer XIO.32
- net PB3: now also J9.12; no longer XIO.31
- net PC0: now also J12.9; no longer XIO.18
- net PC1: now also J9.5; no longer XIO.17
- net PC2: now also J12.10; no longer XIO.16
- net PC3: now also J9.4; no longer XIO.15
- net PC4: now also J12.11; no longer XIO.14
- net PC5: now also J9.3; no longer XIO.13
- net PC6: now also J12.12; no longer XIO.12
- net PC7: now also J9.2; no longer XIO.11
- net PD7: now also J9.6; no longer XIO.19
- net PG0: now also J12.7; no longer XIO.22
- net PG1: now also J9.7; no longer XIO.21
- net PG2: now also J12.8; no longer XIO.20
- net PL0: now also J12.3; no longer XIO.30
- net PL1: now also J9.11; no longer XIO.29
- net PL2: now also J12.4; no longer XIO.28
- net PL3: now also J9.10; no longer XIO.27
- net PL4: now also J12.5; no longer XIO.26
- net PL5: now also J9.9; no longer XIO.25
- net PL6: now also J12.6; no longer XIO.24
- net PL7: now also J9.8; no longer XIO.23
- net RESET: now also R22.1
- net RXD1: now also BLUETOOTH_J6.4; no longer J12.4
- net RXD2: now also IC5.1, RXD2_JUMPER.1; no longer J13.2
- net TXD1: now also BLUETOOTH_J6.5; no longer J12.5
- net TXD2: now also IC5.4, TXD2_JUMPER.1; no longer J13.1
- net V_USB: now also R23.2
Routing:
- net V_USB: track 0.00 -> 47.3 mm, vias 0 -> 2
- net RESET: track 0.00 -> 44.0 mm, vias 0 -> 2
- net PE1: track 0.00 -> 37.8 mm
- net +5V: track 0.00 -> 33.8 mm, vias 0 -> 2
- net PE0: track 0.00 -> 33.4 mm
- net N$9: track 0.00 -> 30.5 mm, vias 0 -> 2
- net N$11: track 0.00 -> 30.4 mm, vias 0 -> 2
- net GND: track 0.00 -> 29.9 mm, vias 0 -> 7
- net FTDI_3.3V: track 0.00 -> 20.2 mm
- net N$4: track 0.00 -> 18.2 mm, vias 0 -> 2
- net USBDP: track 0.00 -> 16.5 mm, vias 0 -> 2
- net USBDN: track 0.00 -> 15.6 mm
- net N$7: track 0.00 -> 13.5 mm
- net FTDI_CBUS1: track 0.00 -> 11.6 mm
- net FTDI_CBUS0: track 0.00 -> 7.30 mm
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- added copper zone on layer 1, net +3V3
- added copper zone on layer 1, net +5V
- added copper zone on layer 16, net GND
Other:
- board text added: "Aground on the FTDI is not connected to anything at the moment"
