File: PowerBoard/Power Supply Board.sch (EAGLE design)
At the start: 37 parts, among them IC3 LM2675

Commit message: Power Supply Board changes
Parts:
- removed X3, X4: (no value), con-wago-500:W237-102
- added U$5, U$6: XT60, HostlerLib:XT60
Connections:
- net 48V+: now also U$5.2, U$6.2; no longer X3-1.KL, X4-1.KL
- net 48V-: now also U$5.1, U$6.1; no longer X3-2.KL, X4-2.KL
Changed lines of the file:
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@@
 <part name="C2" library="SparkFun-Capacitors" deviceset="4.7UF-6.3V-10%(0603)" device="0603" value="4.7uF"/>
 <part name="C6" library="capacitor-wima" deviceset="C" device="2,5-3"/>
-<part name="X3" library="con-wago-500" deviceset="W237-102" device=""/>
-<part name="X4" library="con-wago-500" deviceset="W237-102" device=""/>
 <part name="C7" library="capacitor-wima" deviceset="C" device="2,5-3"/>
 <part name="C8" library="capacitor-wima" deviceset="C" device="2,5-3"/>
@@
 <part name="JP3" library="pinhead" deviceset="PINHD-1X2" device=""/>
 <part name="JP4" library="pinhead" deviceset="PINHD-1X2" device=""/>
+<part name="U$5" library="HostlerLib" deviceset="XT60" device=""/>
+<part name="U$6" library="HostlerLib" deviceset="XT60" device=""/>
 </parts>
 <sheets>
@@
 <instance part="C2" gate="G$1" x="287.02" y="66.04" rot="R90"/>
 <instance part="C6" gate="G$1" x="289.56" y="50.8" rot="MR180"/>
-<instance part="X3" gate="-1" x="78.74" y="99.06"/>
-<instance part="X3" gate="-2" x="78.74" y="91.44"/>
-<instance part="X4" gate="-1" x="78.74" y="58.42"/>
-<instance part="X4" gate="-2" x="78.74" y="50.8"/>
 <instance part="C7" gate="G$1" x="86.36" y="96.52"/>
 <instance part="C8" gate="G$1" x="86.36" y="55.88"/>
@@
 <instance part="JP3" gate="G$1" x="322.58" y="-15.24"/>
 <instance part="JP4" gate="G$1" x="332.74" y="-15.24"/>
+<instance part="U$5" gate="G$1" x="71.12" y="96.52" rot="R180"/>
+<instance part="U$6" gate="G$1" x="68.58" y="55.88" rot="R180"/>
 </instances>
 <busses>
@@
 </segment>
 <segment>
-<wire x1="83.82" y1="99.06" x2="86.36" y2="99.06" width="0.1524" layer="91"/>
 <label x="91.44" y="99.06" size="1.778" layer="95" xref="yes"/>
 <pinref part="C7" gate="G$1" pin="1"/>
 <wire x1="86.36" y1="99.06" x2="91.44" y2="99.06" width="0.1524" layer="91"/>
 <junction x="86.36" y="99.06"/>
-<pinref part="X3" gate="-1" pin="KL"/>
-</segment>
-<segment>
-<wire x1="83.82" y1="58.42" x2="86.36" y2="58.42" width="0.1524" layer="91"/>
+<wire x1="86.36" y1="99.06" x2="81.28" y2="99.06" width="0.1524" layer="91"/>
+<wire x1="81.28" y1="99.06" x2="81.28" y2="96.52" width="0.1524" layer="91"/>
+<pinref part="U$5" gate="G$1" pin="2"/>
+<wire x1="81.28" y1="96.52" x2="73.66" y2="96.52" width="0.1524" layer="91"/>
+</segment>
+<segment>
 <label x="91.44" y="58.42" size="1.778" layer="95" xref="yes"/>
 <pinref part="C8" gate="G$1" pin="1"/>
 <wire x1="86.36" y1="58.42" x2="91.44" y2="58.42" width="0.1524" layer="91"/>
+<wire x1="86.36" y1="58.42" x2="78.74" y2="58.42" width="0.1524" layer="91"/>
 <junction x="86.36" y="58.42"/>
-<pinref part="X4" gate="-1" pin="KL"/>
+<wire x1="78.74" y1="58.42" x2="78.74" y2="55.88" width="0.1524" layer="91"/>
+<pinref part="U$6" gate="G$1" pin="2"/>
+<wire x1="78.74" y1="55.88" x2="71.12" y2="55.88" width="0.1524" layer="91"/>
 </segment>
 </net>
@@
 </segment>
 <segment>
-<wire x1="83.82" y1="91.44" x2="86.36" y2="91.44" width="0.1524" layer="91"/>
 <label x="91.44" y="91.44" size="1.778" layer="95" xref="yes"/>
 <pinref part="C7" gate="G$1" pin="2"/>
 <wire x1="86.36" y1="91.44" x2="91.44" y2="91.44" width="0.1524" layer="91"/>
 <junction x="86.36" y="91.44"/>
-<pinref part="X3" gate="-2" pin="KL"/>
-</segment>
-<segment>
-<wire x1="83.82" y1="50.8" x2="86.36" y2="50.8" width="0.1524" layer="91"/>
+<pinref part="U$5" gate="G$1" pin="1"/>
+<wire x1="73.66" y1="93.98" x2="81.28" y2="93.98" width="0.1524" layer="91"/>
+<wire x1="81.28" y1="93.98" x2="81.28" y2="91.44" width="0.1524" layer="91"/>
+<wire x1="81.28" y1="91.44" x2="86.36" y2="91.44" width="0.1524" layer="91"/>
+</segment>
+<segment>
 <label x="91.44" y="50.8" size="1.778" layer="95" xref="yes"/>
 <pinref part="C8" gate="G$1" pin="2"/>
 <wire x1="86.36" y1="50.8" x2="91.44" y2="50.8" width="0.1524" layer="91"/>
 <junction x="86.36" y="50.8"/>
-<pinref part="X4" gate="-2" pin="KL"/>
-</segment>
-</net>
+<wire x1="86.36" y1="50.8" x2="78.74" y2="50.8" width="0.1524" layer="91"/>
+<wire x1="78.74" y1="50.8" x2="78.74" y2="53.34" width="0.1524" layer="91"/>
+<pinref part="U$6" gate="G$1" pin="1"/>
+<wire x1="78.74" y1="53.34" x2="71.12" y2="53.34" width="0.1524" layer="91"/>
+</segment>
+</net>

Commit message: Power Supply Labeling
Parts:
- added JP5, JP6: (no value), adafruit:PINHD-1X1
- added JP7: (no value), pinhead:PINHD-1X2
Connections:
- net A0: now also JP5.1
- net A1: now also JP6.1
- net GROUNDOUT: now also JP7.2
- net POWER_BANK_0: now also JP7.1
Changed lines of the file:
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@@
 <part name="U$5" library="HostlerLib" deviceset="XT60" device=""/>
 <part name="U$6" library="HostlerLib" deviceset="XT60" device=""/>
+<part name="JP5" library="adafruit" deviceset="PINHD-1X1" device=""/>
+<part name="JP6" library="adafruit" deviceset="PINHD-1X1" device=""/>
+<part name="JP7" library="pinhead" deviceset="PINHD-1X2" device=""/>
 </parts>
 <sheets>
@@
 <instance part="U$5" gate="G$1" x="71.12" y="96.52" rot="R180"/>
 <instance part="U$6" gate="G$1" x="68.58" y="55.88" rot="R180"/>
+<instance part="JP5" gate="G$1" x="297.18" y="119.38"/>
+<instance part="JP6" gate="G$1" x="297.18" y="76.2"/>
+<instance part="JP7" gate="G$1" x="116.84" y="20.32"/>
 </instances>
 <busses>
@@
 <label x="294.64" y="109.22" size="1.778" layer="95" xref="yes"/>
 </segment>
+<segment>
+<wire x1="106.68" y1="20.32" x2="114.3" y2="20.32" width="0.1524" layer="91"/>
+<label x="106.68" y="20.32" size="1.778" layer="95" rot="R180" xref="yes"/>
+<pinref part="JP7" gate="G$1" pin="2"/>
+</segment>
 </net>
 <net name="TM1" class="0">
@@
 <wire x1="279.4" y1="114.3" x2="279.4" y2="119.38" width="0.1524" layer="91"/>
 <wire x1="279.4" y1="119.38" x2="294.64" y2="119.38" width="0.1524" layer="91"/>
+<pinref part="JP5" gate="G$1" pin="1"/>
 </segment>
 </net>
@@
 <wire x1="279.4" y1="71.12" x2="279.4" y2="76.2" width="0.1524" layer="91"/>
 <wire x1="279.4" y1="76.2" x2="294.64" y2="76.2" width="0.1524" layer="91"/>
+<pinref part="JP6" gate="G$1" pin="1"/>
 </segment>
 </net>
@@
 <pinref part="JP2" gate="G$1" pin="1"/>
 </segment>
-</net>
+<segment>
+<wire x1="106.68" y1="22.86" x2="114.3" y2="22.86" width="0.1524" layer="91"/>
+<label x="106.68" y="22.86" size="1.778" layer="95" rot="R180" xref="yes"/>
+<pinref part="JP7" gate="G$1" pin="1"/>
+</segment>
+</net>

Commit message: slight routing additions
Parts:
- added JP8: (no value), pinhead:PINHD-1X2
Connections:
- net GROUNDOUT: now also JP8.2
- net POWER_BANK_0: now also JP8.1
Changed lines of the file:
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@@
 <part name="JP6" library="adafruit" deviceset="PINHD-1X1" device=""/>
 <part name="JP7" library="pinhead" deviceset="PINHD-1X2" device=""/>
+<part name="JP8" library="pinhead" deviceset="PINHD-1X2" device=""/>
 </parts>
 <sheets>
@@
 <instance part="JP6" gate="G$1" x="297.18" y="76.2"/>
 <instance part="JP7" gate="G$1" x="116.84" y="20.32"/>
+<instance part="JP8" gate="G$1" x="154.94" y="20.32"/>
 </instances>
 <busses>
@@
 <wire x1="289.56" y1="48.26" x2="187.96" y2="48.26" width="0.1524" layer="91"/>
 <pinref part="C6" gate="G$1" pin="1"/>
-<pinref part="VC1" gate="G$1" pin="-OUT2"/>
 <wire x1="312.42" y1="91.44" x2="289.56" y2="91.44" width="0.1524" layer="91"/>
 <wire x1="289.56" y1="91.44" x2="187.96" y2="91.44" width="0.1524" layer="91"/>
 <wire x1="187.96" y1="91.44" x2="182.88" y2="91.44" width="0.1524" layer="91"/>
-<wire x1="182.88" y1="91.44" x2="175.26" y2="81.28" width="0.1524" layer="91"/>
 <pinref part="VC1" gate="G$1" pin="-OUT1"/>
 <wire x1="175.26" y1="99.06" x2="177.8" y2="99.06" width="0.1524" layer="91"/>
 <wire x1="177.8" y1="99.06" x2="182.88" y2="91.44" width="0.1524" layer="91"/>
 <label x="293.624" y="89.154" size="1.778" layer="95"/>
-<pinref part="VC2" gate="G$1" pin="-OUT2"/>
 <wire x1="187.96" y1="48.26" x2="185.42" y2="48.26" width="0.1524" layer="91"/>
-<wire x1="185.42" y1="48.26" x2="175.26" y2="38.1" width="0.1524" layer="91"/>
 <pinref part="VC2" gate="G$1" pin="-OUT1"/>
 <wire x1="175.26" y1="55.88" x2="177.8" y2="55.88" width="0.1524" layer="91"/>
@@
 <pinref part="U$4" gate="G$1" pin="2"/>
 <wire x1="320.04" y1="50.8" x2="335.28" y2="50.8" width="0.1524" layer="91"/>
+<pinref part="VC1" gate="G$1" pin="-OUT2"/>
+<wire x1="175.26" y1="81.28" x2="182.88" y2="91.44" width="0.1524" layer="91"/>
+<junction x="182.88" y="91.44"/>
+<pinref part="VC2" gate="G$1" pin="-OUT2"/>
+<wire x1="175.26" y1="38.1" x2="185.42" y2="48.26" width="0.1524" layer="91"/>
+<junction x="185.42" y="48.26"/>
 </segment>
 <segment>
@@
 <pinref part="JP7" gate="G$1" pin="2"/>
 </segment>
+<segment>
+<wire x1="144.78" y1="20.32" x2="152.4" y2="20.32" width="0.1524" layer="91"/>
+<label x="144.78" y="20.32" size="1.778" layer="95" rot="R180" xref="yes"/>
+<pinref part="JP8" gate="G$1" pin="2"/>
+</segment>
 </net>
 <net name="TM1" class="0">
@@
 <pinref part="JP7" gate="G$1" pin="1"/>
 </segment>
+<segment>
+<wire x1="144.78" y1="22.86" x2="152.4" y2="22.86" width="0.1524" layer="91"/>
+<label x="144.78" y="22.86" size="1.778" layer="95" rot="R180" xref="yes"/>
+<pinref part="JP8" gate="G$1" pin="1"/>
+</segment>
 </net>
 <net name="FUSE2IN" class="0">
@@
 <net name="BUCK1OUT" class="0">
 <segment>
+<pinref part="CSENSE1" gate="G$1" pin="IP+@2"/>
+<wire x1="236.22" y1="71.12" x2="238.76" y2="71.12" width="0.1524" layer="91"/>
+<pinref part="CSENSE1" gate="G$1" pin="IP+@1"/>
+<wire x1="238.76" y1="73.66" x2="236.22" y2="73.66" width="0.1524" layer="91"/>
+<wire x1="236.22" y1="73.66" x2="236.22" y2="71.12" width="0.1524" layer="91"/>
+<junction x="236.22" y="73.66"/>
+<wire x1="193.04" y1="73.66" x2="236.22" y2="73.66" width="0.1524" layer="91"/>
 <pinref part="VC2" gate="G$1" pin="+OUT2"/>
 <wire x1="175.26" y1="48.26" x2="177.8" y2="48.26" width="0.1524" layer="91"/>
@@
 <junction x="185.42" y="55.88"/>
 <wire x1="185.42" y1="55.88" x2="193.04" y2="55.88" width="0.1524" layer="91"/>
+<label x="198.12" y="55.88" size="1.778" layer="95" xref="yes"/>
+<wire x1="193.04" y1="55.88" x2="198.12" y2="55.88" width="0.1524" layer="91"/>
 <wire x1="193.04" y1="73.66" x2="193.04" y2="55.88" width="0.1524" layer="91"/>
 <junction x="193.04" y="55.88"/>
-<wire x1="193.04" y1="55.88" x2="198.12" y2="55.88" width="0.1524" layer="91"/>
-<label x="198.12" y="55.88" size="1.778" layer="95" xref="yes"/>
-</segment>
-<segment>
-<pinref part="CSENSE1" gate="G$1" pin="IP+@2"/>
-<wire x1="236.22" y1="71.12" x2="238.76" y2="71.12" width="0.1524" layer="91"/>
-<pinref part="CSENSE1" gate="G$1" pin="IP+@1"/>
-<wire x1="238.76" y1="73.66" x2="236.22" y2="73.66" width="0.1524" layer="91"/>
-<wire x1="236.22" y1="73.66" x2="236.22" y2="71.12" width="0.1524" layer="91"/>
-<junction x="236.22" y="73.66"/>
-<wire x1="193.04" y1="73.66" x2="236.22" y2="73.66" width="0.1524" layer="91"/>
 </segment>
 </net>
@@
 </sheet>
 </sheets>
+<errors>
+</errors>
 </schematic>
 </drawing>

Commit message: Power gerber generated
Connections:
- removed net PC2: SV2.1, SV2.2, VC2.PC
- net PC1: now also SV2.1, SV2.2, VC2.PC
Changed lines of the file:
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@@
 <wire x1="142.24" y1="91.44" x2="139.7" y2="91.44" width="0.1524" layer="91"/>
+</segment>
+<segment>
+<pinref part="SV2" gate="1" pin="2"/>
+<pinref part="VC2" gate="G$1" pin="PC"/>
+<wire x1="139.7" y1="50.8" x2="142.24" y2="50.8" width="0.1524" layer="91"/>
+<wire x1="142.24" y1="50.8" x2="142.24" y2="48.26" width="0.1524" layer="91"/>
+<junction x="142.24" y="50.8"/>
+<pinref part="SV2" gate="1" pin="1"/>
+<wire x1="142.24" y1="48.26" x2="139.7" y2="48.26" width="0.1524" layer="91"/>
 </segment>
 </net>
@@
 </segment>
 </net>
-<net name="PC2" class="0">
-<segment>
-<pinref part="SV2" gate="1" pin="2"/>
-<pinref part="VC2" gate="G$1" pin="PC"/>
-<wire x1="139.7" y1="50.8" x2="142.24" y2="50.8" width="0.1524" layer="91"/>
-<wire x1="142.24" y1="50.8" x2="142.24" y2="48.26" width="0.1524" layer="91"/>
-<junction x="142.24" y="50.8"/>
-<pinref part="SV2" gate="1" pin="1"/>
-<wire x1="142.24" y1="48.26" x2="139.7" y2="48.26" width="0.1524" layer="91"/>
-</segment>
-</net>

Commit message: final changes for FAB
Changed lines of the file:
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@@
 <instance part="C3" gate="A" x="129.54" y="-15.24" smashed="yes" rot="R90">
 <attribute name="NAME" x="123.9774" y="-19.9644" size="2.0828" layer="95" ratio="6" rot="SR90"/>
-<attribute name="VALUE" x="123.7234" y="-14.5034" size="2.0828" layer="96" ratio="6" rot="SR90"/>
+<attribute name="VALUE" x="123.7234" y="-11.9634" size="2.0828" layer="96" ratio="6" rot="SR90"/>
 </instance>
 <instance part="C11" gate="A" x="139.7" y="-15.24" smashed="yes" rot="R90">
 <attribute name="NAME" x="135.6614" y="-19.9644" size="2.0828" layer="95" ratio="6" rot="SR90"/>
-<attribute name="VALUE" x="135.6614" y="-15.5194" size="2.0828" layer="96" ratio="6" rot="SR90"/>
+<attribute name="VALUE" x="135.6614" y="-12.9794" size="2.0828" layer="96" ratio="6" rot="SR90"/>
 </instance>
 <instance part="C12" gate="A" x="149.86" y="-15.24" smashed="yes" rot="R90">
 <attribute name="NAME" x="145.8214" y="-20.9804" size="2.0828" layer="95" ratio="6" rot="SR90"/>
-<attribute name="VALUE" x="145.8214" y="-16.5354" size="2.0828" layer="96" ratio="6" rot="SR90"/>
+<attribute name="VALUE" x="145.8214" y="-13.9954" size="2.0828" layer="96" ratio="6" rot="SR90"/>
 </instance>
 <instance part="SUPPLY2" gate="GND" x="203.2" y="-30.48"/>
@@
 <instance part="U$4" gate="G$1" x="337.82" y="50.8"/>
 <instance part="C15" gate="A" x="309.88" y="71.12" smashed="yes" rot="R90">
-<attribute name="NAME" x="305.8414" y="65.3796" size="2.0828" layer="95" ratio="6" rot="SR90"/>
+<attribute name="NAME" x="316.0014" y="72.9996" size="2.0828" layer="95" ratio="6" rot="SR90"/>
 <attribute name="VALUE" x="305.8414" y="69.8246" size="2.0828" layer="96" ratio="6" rot="SR90"/>
 </instance>
 <instance part="C16" gate="A" x="309.88" y="114.3" smashed="yes" rot="R90">
-<attribute name="NAME" x="305.8414" y="108.5596" size="2.0828" layer="95" ratio="6" rot="SR90"/>
+<attribute name="NAME" x="316.0014" y="116.1796" size="2.0828" layer="95" ratio="6" rot="SR90"/>
 <attribute name="VALUE" x="305.8414" y="113.0046" size="2.0828" layer="96" ratio="6" rot="SR90"/>
 </instance>
